File: USB-DAC-PCM2902.sch (KiCad schematic (older format))
At the start: 25 parts

Commit message: update, draft route done,
Parts:
- C1, C10, C11, C2, C4, C6, C8, C9: renamed from C?; footprint (none) -> Capacitor_SMD:CP_Elec_4x5.3
- C3, C5, C7: renamed from C?; footprint (none) -> Capacitor_SMD:C_0603_1608Metric_Pad1.05x0.95mm_HandSolder
- D1: renamed from D?; footprint (none) -> LED_SMD:LED_0603_1608Metric_Pad1.05x0.95mm_HandSolder
- J1: renamed from J?; footprint (none) -> Connector_PinHeader_1.27mm:PinHeader_1x02_P1.27mm_Vertical
- J2: renamed from J?; footprint (none) -> Connector_Audio:Jack_3.5mm_PJ320D_Horizontal
- R1, R2, R3, R4, R5, R6, R7: renamed from R?; footprint (none) -> Resistor_SMD:R_0603_1608Metric_Pad1.05x0.95mm_HandSolder
- U1: renamed from U?; footprint (none) -> footprint-lib:usb-PCB
- U2: renamed from U?; footprint (none) -> Package_SO:SSOP-28_3.9x9.9mm_P0.635mm
- U3: renamed from U?; footprint (none) -> Package_SO:SSOP-8_2.95x2.8mm_P0.65mm
- Y1: renamed from Y?; footprint (none) -> w_crystal:crystal_hc-49s

Commit message: update vol button,
Parts:
- added SW1: MUTE, Button_Switch_THT:SW_PUSH_6mm_H4.3mm, symbol Switch:SW_Push_45deg
- added SW2: VOL_DOWN, Button_Switch_THT:SW_PUSH_6mm_H4.3mm, symbol Switch:SW_Push_45deg
- added SW3: VOL_UP, Button_Switch_THT:SW_PUSH_6mm_H4.3mm, symbol Switch:SW_Push_45deg
Connections:
- net labels added: PIN28, VOL_DOWN, VOL_MUTE, VOL_UP
- wire segments 112 -> 122
Changed lines of the file:
@@
 EESchema Schematic File Version 4
+LIBS:USB-DAC-PCM2902-cache
 EELAYER 26 0
 EELAYER END
@@
 	5700 2750 5700 2850
 Wire Wire Line
-	5700 1650 7650 1650
-Wire Wire Line
-	7650 1650 7650 2150
-Wire Wire Line
-	7650 2150 7400 2150
+	5700 1650 8000 1650
+Wire Wire Line
+	8000 1650 8000 2150
+Wire Wire Line
+	8000 2150 7400 2150
 Connection ~ 5700 1650
 $Comp
@@
 	7400 2550 8050 2550
 Wire Wire Line
-	7650 2150 8050 2150
-Connection ~ 7650 2150
+	8000 2150 8050 2150
+Connection ~ 8000 2150
 $Comp
 L Connector_Generic:Conn_01x02 J1
@@
 Wire Wire Line
 	4700 2950 5400 2950
+$Comp
+L Switch:SW_Push_45deg SW1
+U 1 1 5BF5E46A
+P 4100 800
+F 0 "SW1" V 4150 950 50  0000 L CNN
+F 1 "MUTE" V 4100 950 50  0000 L CNN
+F 2 "Button_Switch_THT:SW_PUSH_6mm_H4.3mm" H 4100 800 50  0001 C CNN
+F 3 "" H 4100 800 50  0001 C CNN
+	1    4100 800
+	0    1    -1   0
+$EndComp
+$Comp
+L Switch:SW_Push_45deg SW2
+U 1 1 5BF5E754
+P 4100 1050
+F 0 "SW2" V 4150 900 50  0000 R CNN
+F 1 "VOL_DOWN" V 4100 900 50  0000 R CNN
+F 2 "Button_Switch_THT:SW_PUSH_6mm_H4.3mm" H 4100 1050 50  0001 C CNN
+F 3 "" H 4100 1050 50  0001 C CNN
+	1    4100 1050
+	0    1    -1   0
+$EndComp
+$Comp
+L Switch:SW_Push_45deg SW3
+U 1 1 5BF5EB5C
+P 4100 1300
+F 0 "SW3" V 4150 1150 50  0000 R CNN
+F 1 "VOL_UP" V 4100 1150 50  0000 R CNN
+F 2 "Button_Switch_THT:SW_PUSH_6mm_H4.3mm" H 4100 1300 50  0001 C CNN
+F 3 "" H 4100 1300 50  0001 C CNN
+	1    4100 1300
+	0    1    -1   0
+$EndComp
+Text Label 7750 2050 2    50   ~ 0
+PIN28
+Wire Wire Line
+	7750 2050 7400 2050
+Text Label 3250 700  0    50   ~ 0
+PIN28
+Wire Wire Line
+	3250 700  4000 700
+Wire Wire Line
+	4000 700  4000 950
+Connection ~ 4000 700
+Connection ~ 4000 950
+Wire Wire Line
+	4000 950  4000 1200
+Text Label 5200 2650 0    50   ~ 0
+VOL_UP
+Text Label 5200 2550 0    50   ~ 0
+VOL_DOWN
+Text Label 5200 2450 0    50   ~ 0
+VOL_MUTE
+Wire Wire Line
+	5200 2450 5950 2450
+Wire Wire Line
+	5950 2550 5200 2550
+Wire Wire Line
+	5200 2650 5950 2650
+Text Label 4950 1400 2    50   ~ 0
+VOL_UP
+Text Label 4950 1150 2    50   ~ 0
+VOL_DOWN
+Text Label 4950 900  2    50   ~ 0
+VOL_MUTE
+Wire Wire Line
+	4950 900  4200 900
+Wire Wire Line
+	4200 1150 4950 1150
+Wire Wire Line
+	4950 1400 4200 1400
 $EndSCHEMATC

Commit message: update,
Parts:
- added H1, H2, H3, H4: MOUNT_M3, MountingHole:MountingHole_3.2mm_M3_DIN965, symbol taobao-mounting-hole:MOUNT_M3
Changed lines of the file:
@@
 Wire Wire Line
 	4950 1400 4200 1400
+$Comp
+L taobao-mounting-hole:MOUNT_M3 H1
+U 1 1 5BF85F10
+P 5900 6750
+F 0 "H1" H 6000 6796 50  0000 L CNN
+F 1 "MOUNT_M3" H 6000 6705 50  0000 L CNN
+F 2 "MountingHole:MountingHole_3.2mm_M3_DIN965" H 5900 6750 50  0001 C CNN
+F 3 "~" H 5900 6750 50  0001 C CNN
+	1    5900 6750
+	1    0    0    -1
+$EndComp
+$Comp
+L taobao-mounting-hole:MOUNT_M3 H2
+U 1 1 5BF85F64
+P 5900 6950
+F 0 "H2" H 6000 6996 50  0000 L CNN
+F 1 "MOUNT_M3" H 6000 6905 50  0000 L CNN
+F 2 "MountingHole:MountingHole_3.2mm_M3_DIN965" H 5900 6950 50  0001 C CNN
+F 3 "~" H 5900 6950 50  0001 C CNN
+	1    5900 6950
+	1    0    0    -1
+$EndComp
+$Comp
+L taobao-mounting-hole:MOUNT_M3 H3
+U 1 1 5BF85FB6
+P 5900 7150
+F 0 "H3" H 6000 7196 50  0000 L CNN
+F 1 "MOUNT_M3" H 6000 7105 50  0000 L CNN
+F 2 "MountingHole:MountingHole_3.2mm_M3_DIN965" H 5900 7150 50  0001 C CNN
+F 3 "~" H 5900 7150 50  0001 C CNN
+	1    5900 7150
+	1    0    0    -1
+$EndComp
+$Comp
+L taobao-mounting-hole:MOUNT_M3 H4
+U 1 1 5BF86008
+P 5900 7350
+F 0 "H4" H 6000 7396 50  0000 L CNN
+F 1 "MOUNT_M3" H 6000 7305 50  0000 L CNN
+F 2 "MountingHole:MountingHole_3.2mm_M3_DIN965" H 5900 7350 50  0001 C CNN
+F 3 "~" H 5900 7350 50  0001 C CNN
+	1    5900 7350
+	1    0    0    -1
+$EndComp
 $EndSCHEMATC
