File: USB-DAC-PCM2902.sch (KiCad schematic (older format))
At the start: 32 parts, among them J1 Conn_01x02, J2 PJ-320D, SW1 MUTE, SW2 VOL_DOWN, SW3 VOL_UP, U1 USB_PCB, U2 PCM2902, U3 LP2951CM, Y1 O12M

Commit message: upadte,
Parts:
- H1, H2, H3, H4: footprint MountingHole:MountingHole_3.2mm_M3_DIN965 -> MountingHole:MountingHole_2.2mm_M2_DIN965
- J1: footprint Connector_PinHeader_1.27mm:PinHeader_1x02_P1.27mm_Vertical -> Connector_PinHeader_2.54mm:PinHeader_1x02_P2.54mm_Vertical
- J2: footprint Connector_Audio:Jack_3.5mm_PJ320D_Horizontal -> footprint-lib:PJ320D_3.5mm_Jack
Changed lines of the file:
@@
 F 0 "J1" H 9000 2250 50  0000 L CNN
 F 1 "Conn_01x02" H 9000 2150 50  0000 L CNN
-F 2 "Connector_PinHeader_1.27mm:PinHeader_1x02_P1.27mm_Vertical" H 8900 2250 50  0001 C CNN
+F 2 "Connector_PinHeader_2.54mm:PinHeader_1x02_P2.54mm_Vertical" H 8900 2250 50  0001 C CNN
 F 3 "~" H 8900 2250 50  0001 C CNN
 	1    8900 2250
@@
 F 0 "J2" H 7200 4350 50  0000 C CNN
 F 1 "PJ-320D" H 7200 4450 50  0000 C CNN
-F 2 "Connector_Audio:Jack_3.5mm_PJ320D_Horizontal" H 6900 4750 50  0001 C CNN
+F 2 "footprint-lib:PJ320D_3.5mm_Jack" H 6900 4750 50  0001 C CNN
 F 3 "" H 6900 4750 50  0000 C CNN
 	1    7100 4750
@@
 F 0 "H1" H 6000 6796 50  0000 L CNN
 F 1 "MOUNT_M3" H 6000 6705 50  0000 L CNN
-F 2 "MountingHole:MountingHole_3.2mm_M3_DIN965" H 5900 6750 50  0001 C CNN
+F 2 "MountingHole:MountingHole_2.2mm_M2_DIN965" H 5900 6750 50  0001 C CNN
 F 3 "~" H 5900 6750 50  0001 C CNN
 	1    5900 6750
@@
 F 0 "H2" H 6000 6996 50  0000 L CNN
 F 1 "MOUNT_M3" H 6000 6905 50  0000 L CNN
-F 2 "MountingHole:MountingHole_3.2mm_M3_DIN965" H 5900 6950 50  0001 C CNN
+F 2 "MountingHole:MountingHole_2.2mm_M2_DIN965" H 5900 6950 50  0001 C CNN
 F 3 "~" H 5900 6950 50  0001 C CNN
 	1    5900 6950
@@
 F 0 "H3" H 6000 7196 50  0000 L CNN
 F 1 "MOUNT_M3" H 6000 7105 50  0000 L CNN
-F 2 "MountingHole:MountingHole_3.2mm_M3_DIN965" H 5900 7150 50  0001 C CNN
+F 2 "MountingHole:MountingHole_2.2mm_M2_DIN965" H 5900 7150 50  0001 C CNN
 F 3 "~" H 5900 7150 50  0001 C CNN
 	1    5900 7150
@@
 F 0 "H4" H 6000 7396 50  0000 L CNN
 F 1 "MOUNT_M3" H 6000 7305 50  0000 L CNN
-F 2 "MountingHole:MountingHole_3.2mm_M3_DIN965" H 5900 7350 50  0001 C CNN
+F 2 "MountingHole:MountingHole_2.2mm_M2_DIN965" H 5900 7350 50  0001 C CNN
 F 3 "~" H 5900 7350 50  0001 C CNN
 	1    5900 7350
@@
 Data
 89 50 4E 47 0D 0A 1A 0A 00 00 00 0D 49 48 44 52 00 00 02 BC 00 00 01 68 08 02 00 00 00 3A 9F BF
-B0 00 00 00 03 73 42 49 54 08 08 08 DB E1 4F E0 00 00 00 09 70 48 59 73 00 00 0B 12 00 00 0B 12
-01 D2 DD 7E FC 00 00 20 00 49 44 41 54 78 9C EC BD 67 70 5C D7 79 3E 7E CE 2D DB 2B B0 00 76 81
+B0 00 00 00 03 73 42 49 54 08 08 08 DB E1 4F E0 00 00 00 09 70 48 59 73 00 00 0A F0 00 00 0A F0
+01 42 AC 34 98 00 00 20 00 49 44 41 54 78 9C EC BD 67 70 5C D7 79 3E 7E CE 2D DB 2B B0 00 76 81
 DD 45 25 0A 49 B0 77 51 14 C5 A2 4E 4B 96 64 5B B6 14 3B 1E DB 33 76 66 EC 19 27 13 7F C8 FC 32
 FF D8 1F 32 F9 94 D8 F1 D8 33 8A E3 12 5B 4A 24 AB 99 14 45 51 B2 28 51 24 25 52 2C 60 07 C0 82

Commit message: upadte,
Parts:
- SW2: value VOL_DOWN -> DOWN
- SW3: value VOL_UP -> UP
Changed lines of the file:
@@
 P 4100 1050
 F 0 "SW2" V 4150 900 50  0000 R CNN
-F 1 "VOL_DOWN" V 4100 900 50  0000 R CNN
+F 1 "DOWN" V 4100 900 50  0000 R CNN
 F 2 "Button_Switch_THT:SW_PUSH_6mm_H4.3mm" H 4100 1050 50  0001 C CNN
 F 3 "" H 4100 1050 50  0001 C CNN
@@
 P 4100 1300
 F 0 "SW3" V 4150 1150 50  0000 R CNN
-F 1 "VOL_UP" V 4100 1150 50  0000 R CNN
+F 1 "UP" V 4100 1150 50  0000 R CNN
 F 2 "Button_Switch_THT:SW_PUSH_6mm_H4.3mm" H 4100 1300 50  0001 C CNN
 F 3 "" H 4100 1300 50  0001 C CNN
