File: USB-DAC-PCM2902.sch (KiCad schematic (older format))
At the start: 32 parts, among them J1 Conn_01x02, J2 PJ-320D, SW1 MUTE, SW2 VOL_DOWN, SW3 VOL_UP, U1 USB_PCB, U2 PCM2902, U3 LP2951CM, Y1 O12M

Commit message: update,
Parts:
- J1: footprint Connector_PinHeader_1.27mm:PinHeader_1x02_P1.27mm_Vertical -> Connector_PinHeader_2.54mm:PinHeader_1x02_P2.54mm_Vertical
Changed lines of the file:
@@
 F 0 "J1" H 9000 2250 50  0000 L CNN
 F 1 "Conn_01x02" H 9000 2150 50  0000 L CNN
-F 2 "Connector_PinHeader_1.27mm:PinHeader_1x02_P1.27mm_Vertical" H 8900 2250 50  0001 C CNN
+F 2 "Connector_PinHeader_2.54mm:PinHeader_1x02_P2.54mm_Vertical" H 8900 2250 50  0001 C CNN
 F 3 "~" H 8900 2250 50  0001 C CNN
 	1    8900 2250
@@
 Data
 89 50 4E 47 0D 0A 1A 0A 00 00 00 0D 49 48 44 52 00 00 02 BC 00 00 01 68 08 02 00 00 00 3A 9F BF
-B0 00 00 00 03 73 42 49 54 08 08 08 DB E1 4F E0 00 00 00 09 70 48 59 73 00 00 0B 12 00 00 0B 12
-01 D2 DD 7E FC 00 00 20 00 49 44 41 54 78 9C EC BD 67 70 5C D7 79 3E 7E CE 2D DB 2B B0 00 76 81
+B0 00 00 00 03 73 42 49 54 08 08 08 DB E1 4F E0 00 00 00 09 70 48 59 73 00 00 0A F0 00 00 0A F0
+01 42 AC 34 98 00 00 20 00 49 44 41 54 78 9C EC BD 67 70 5C D7 79 3E 7E CE 2D DB 2B B0 00 76 81
 DD 45 25 0A 49 B0 77 51 14 C5 A2 4E 4B 96 64 5B B6 14 3B 1E DB 33 76 66 EC 19 27 13 7F C8 FC 32
 FF D8 1F 32 F9 94 D8 F1 D8 33 8A E3 12 5B 4A 24 AB 99 14 45 51 B2 28 51 24 25 52 2C 60 07 C0 82

Commit message: update,
Parts:
- removed R5: R106,0603, Resistor_SMD:R_0603_1608Metric_Pad1.05x0.95mm_HandSolder, symbol taobao-r:R106,0603
Changed lines of the file:
@@
 L taobao-osc:O12M Y1
 U 1 1 5BF62F5E
-P 9000 2800
-F 0 "Y1" V 8950 2900 50  0000 L CNN
-F 1 "O12M" V 9000 2900 50  0000 L CNN
-F 2 "w_crystal:crystal_hc-49s" H 9000 2800 50  0001 C CNN
-F 3 "~" H 9000 2800 50  0001 C CNN
-	1    9000 2800
+P 9350 2800
+F 0 "Y1" V 9304 2712 50  0000 R CNN
+F 1 "O12M" V 9395 2712 50  0000 R CNN
+F 2 "w_crystal:crystal_hc-49s" H 9350 2800 50  0001 C CNN
+F 3 "~" H 9350 2800 50  0001 C CNN
+	1    9350 2800
 	0    -1   1    0
-$EndComp
-$Comp
-L taobao-r:R106,0603 R5
-U 1 1 5BF63130
-P 8800 2800
-F 0 "R5" H 8900 2850 50  0000 L CNN
-F 1 "R106,0603" H 8900 2800 50  0000 L CNN
-F 2 "Resistor_SMD:R_0603_1608Metric_Pad1.05x0.95mm_HandSolder" H 8800 2800 50  0001 C CNN
-F 3 "~" H 8800 2800 50  0001 C CNN
-	1    8800 2800
-	1    0    0    -1
 $EndComp
 $Comp
 L taobao-c:C22pf,0603 C3
 U 1 1 5BF6375A
-P 9250 2950
-F 0 "C3" V 9000 2950 50  0000 C CNN
-F 1 "C22pf,0603" V 9100 2950 50  0000 C CNN
-F 2 "Capacitor_SMD:C_0603_1608Metric_Pad1.05x0.95mm_HandSolder" H 9250 2950 50  0001 C CNN
-F 3 "~" H 9250 2950 50  0001 C CNN
-	1    9250 2950
+P 9600 2950
+F 0 "C3" V 9737 2950 50  0000 C CNN
+F 1 "C22pf,0603" V 9828 2950 50  0000 C CNN
+F 2 "Capacitor_SMD:C_0603_1608Metric_Pad1.05x0.95mm_HandSolder" H 9600 2950 50  0001 C CNN
+F 3 "~" H 9600 2950 50  0001 C CNN
+	1    9600 2950
 	0    1    1    0
 $EndComp
@@
 L taobao-c:C22pf,0603 C5
 U 1 1 5BF637E8
-P 9250 2650
-F 0 "C5" V 9400 2650 50  0000 C CNN
-F 1 "C22pf,0603" V 9500 2650 50  0000 C CNN
-F 2 "Capacitor_SMD:C_0603_1608Metric_Pad1.05x0.95mm_HandSolder" H 9250 2650 50  0001 C CNN
-F 3 "~" H 9250 2650 50  0001 C CNN
-	1    9250 2650
+P 9600 2650
+F 0 "C5" V 9371 2650 50  0000 C CNN
+F 1 "C22pf,0603" V 9462 2650 50  0000 C CNN
+F 2 "Capacitor_SMD:C_0603_1608Metric_Pad1.05x0.95mm_HandSolder" H 9600 2650 50  0001 C CNN
+F 3 "~" H 9600 2650 50  0001 C CNN
+	1    9600 2650
 	0    1    1    0
 $EndComp
 Wire Wire Line
-	9150 2650 9000 2650
+	9500 2650 9350 2650
 Wire Wire Line
 	8800 2650 8800 2700
 Wire Wire Line
-	9000 2700 9000 2650
-Connection ~ 9000 2650
+	9350 2700 9350 2650
+Connection ~ 9350 2650
 Wire Wire Line
-	9000 2650 8800 2650
+	9350 2650 9150 2650
 Wire Wire Line
 	8800 2900 8800 2950
 Wire Wire Line
-	8800 2950 9000 2950
+	9150 2950 9350 2950
 Wire Wire Line
-	9000 2900 9000 2950
-Connection ~ 9000 2950
+	9350 2900 9350 2950
+Connection ~ 9350 2950
 Wire Wire Line
-	9000 2950 9150 2950
+	9350 2950 9500 2950
 Wire Wire Line
-	9350 2650 9500 2650
+	9700 2650 9850 2650
 Wire Wire Line
-	9500 2650 9500 2800
+	9850 2650 9850 2800
 Wire Wire Line
-	9500 2950 9350 2950
+	9850 2950 9700 2950
 $Comp
 L power:GND #PWR0109
 U 1 1 5BF69C59
-P 9700 2950
-F 0 "#PWR0109" H 9700 2700 50  0001 C CNN
-F 1 "GND" H 9750 2750 50  0000 C CNN
-F 2 "" H 9700 2950 50  0001 C CNN
-F 3 "" H 9700 2950 50  0001 C CNN
-	1    9700 2950
+P 10050 2950
+F 0 "#PWR0109" H 10050 2700 50  0001 C CNN
+F 1 "GND" H 10100 2750 50  0000 C CNN
+F 2 "" H 10050 2950 50  0001 C CNN
+F 3 "" H 10050 2950 50  0001 C CNN
+	1    10050 2950
 	1    0    0    -1
 $EndComp
 Wire Wire Line
-	9700 2950 9700 2800
+	10050 2950 10050 2800
 Wire Wire Line
-	9700 2800 9500 2800
-Connection ~ 9500 2800
+	10050 2800 9850 2800
+Connection ~ 9850 2800
 Wire Wire Line
-	9500 2800 9500 2950
+	9850 2800 9850 2950
 Wire Wire Line
 	7400 2750 8600 2750
@@
 Wire Wire Line
 	8600 2650 8800 2650
-Connection ~ 8800 2650
 Wire Wire Line
 	7400 2850 8600 2850
@@
 Wire Wire Line
 	8600 2950 8800 2950
-Connection ~ 8800 2950
 Wire Wire Line
 	8250 2950 8400 2950
