File: USB-DAC-PCM2902.kicad_pcb (KiCad board)
At the start: 2 copper layers, 63 x 34.8 mm, 32 parts, among them J1 Conn_01x02, J2 PJ-320D, SW1 MUTE, SW2 VOL_DOWN, SW3 VOL_UP, U1 USB_PCB, U2 PCM2902, U3 LP2951CM, Y1 O12M

Commit message: upadte,
Parts:
- H2, H3, H4: footprint MountingHole:MountingHole_3.2mm_M3_DIN965 -> MountingHole:MountingHole_2.2mm_M2_DIN965
- J2: footprint Connector_Audio:Jack_3.5mm_PJ320D_Horizontal -> footprint-lib:PJ320D_3.5mm_Jack
Routing:
- net GND: track 169.5 -> 176.6 mm
- net /OUTL: track 27.8 -> 23.6 mm
- net /OUTR: track 18.2 -> 17.7 mm

Commit message: upadte,
Parts:
- SW2: value VOL_DOWN -> DOWN
- SW3: value VOL_UP -> UP
- moved H3 82.8 mm to (20.9, 2.40)
- moved H2 76.8 mm to (20.4, 32.3)
- moved H4 62.1 mm to (41.3, 31.5)
- moved J1 4.00 mm to (60.3, 6.04)
- moved R7 2.87 mm to (24.8, 21.0)
- moved R6 2.77 mm to (22.3, 23.9)
- moved C7 2.76 mm to (24.6, 23.9)
- moved C9 2.24 mm to (17.6, 26.6)
- moved C10 2.00 mm to (24.7, 26.6)
- moved Y1 1.00 mm to (52.5, 7.36)
Routing:
- net /OUTR: track 17.7 -> 27.7 mm, vias 0 -> 2
- net Net-(J1-Pad2): track 33.0 -> 25.5 mm
- net /OUTL: track 23.6 -> 31.0 mm, vias 0 -> 2
- net Net-(R4-Pad2): track 62.8 -> 68.7 mm
- net Net-(C5-Pad2): track 32.6 -> 28.4 mm
- net /VOL_DOWN: track 44.6 -> 40.5 mm
- net Net-(R2-Pad1): track 22.6 -> 19.7 mm
- net Net-(C6-Pad1): track 28.3 -> 31.2 mm, vias 0 -> 2
- net /VOL_UP: track 54.3 -> 51.5 mm
- net /VOL_MUTE: track 30.1 -> 27.4 mm
- net Net-(C7-Pad1): track 31.8 -> 34.5 mm
- net Net-(C4-Pad1): track 16.1 -> 13.6 mm
- net Net-(C7-Pad2): track 7.50 -> 9.85 mm
- net Net-(R3-Pad1): track 23.9 -> 22.1 mm
- net GND: track 176.6 -> 174.9 mm
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Other:
- board text added: "PCM2902 EVALUATION BOARD 20181126 print1"
- board text removed: "PCM2902 EVALUATION BOARD"
